File: pcb/encoder_key.kicad_sch (KiCad schematic)
At the start: 4 parts, among them SW1 EC11 or MX

Commit message: Increase polling frequency of NKRO report
Parts:
- D1: footprint agausmann:1N4148_Hybrid_SMD_THT -> Diode_THT:D_DO-34_SOD68_P7.62mm_Horizontal
- R10, R9: footprint agausmann:R_Hybrid_SMD_THT -> Resistor_THT:R_Axial_DIN0204_L3.6mm_D1.6mm_P7.62mm_Horizontal
Changed lines of the file:
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@@
     (property "Reference" "D1" (id 0) (at 118.11 69.85 0))
     (property "Value" "1N4148" (id 1) (at 118.11 72.39 0))
-    (property "Footprint" "agausmann:1N4148_Hybrid_SMD_THT" (id 2) (at 118.11 76.2 0)
+    (property "Footprint" "Diode_THT:D_DO-34_SOD68_P7.62mm_Horizontal" (id 2) (at 118.11 76.2 0)
       (effects (font (size 1.27 1.27)) hide)
     )
@@
       (effects (font (size 1.27 1.27)) (justify right))
     )
-    (property "Footprint" "agausmann:R_Hybrid_SMD_THT" (id 2) (at 93.98 69.85 0)
+    (property "Footprint" "Resistor_THT:R_Axial_DIN0204_L3.6mm_D1.6mm_P7.62mm_Horizontal" (id 2) (at 93.98 69.85 0)
       (effects (font (size 1.27 1.27)) hide)
     )
@@
       (effects (font (size 1.27 1.27)) (justify right))
     )
-    (property "Footprint" "agausmann:R_Hybrid_SMD_THT" (id 2) (at 85.09 69.85 0)
+    (property "Footprint" "Resistor_THT:R_Axial_DIN0204_L3.6mm_D1.6mm_P7.62mm_Horizontal" (id 2) (at 85.09 69.85 0)
       (effects (font (size 1.27 1.27)) hide)
     )
