File: pcb/key.kicad_sch (KiCad schematic)
At the start: 2 parts, among them SW7 MX

Commit message: Increase polling frequency of NKRO report
Parts:
- D7: footprint agausmann:1N4148_Hybrid_SMD_THT -> Diode_THT:D_DO-34_SOD68_P7.62mm_Horizontal
Changed lines of the file:
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@@
     (property "Reference" "D7" (id 0) (at 111.76 62.23 0))
     (property "Value" "1N4148" (id 1) (at 111.76 64.77 0))
-    (property "Footprint" "agausmann:1N4148_Hybrid_SMD_THT" (id 2) (at 111.76 68.58 0)
+    (property "Footprint" "Diode_THT:D_DO-34_SOD68_P7.62mm_Horizontal" (id 2) (at 111.76 68.58 0)
       (effects (font (size 1.27 1.27)) hide)
     )
