File: pcb/leds.kicad_sch (KiCad schematic)
At the start: 4 parts, among them U2 MAX6969ANG+, U3 HDSP-521A

Commit message: Increase polling frequency of NKRO report
Parts:
- R11: footprint agausmann:R_Hybrid_SMD_THT -> Resistor_THT:R_Axial_DIN0204_L3.6mm_D1.6mm_P7.62mm_Horizontal
Changed lines of the file:
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@@
       (effects (font (size 1.27 1.27)) (justify left))
     )
-    (property "Footprint" "agausmann:R_Hybrid_SMD_THT" (id 2) (at 66.04 92.71 0)
+    (property "Footprint" "Resistor_THT:R_Axial_DIN0204_L3.6mm_D1.6mm_P7.62mm_Horizontal" (id 2) (at 66.04 92.71 0)
       (effects (font (size 1.27 1.27)) hide)
     )
