File: pcb/matrix.kicad_sch (KiCad schematic)
At the start: 6 parts

Commit message: Increase polling frequency of NKRO report
Parts:
- R1, R2, R3, R4, R5, R6: footprint agausmann:R_Hybrid_SMD_THT -> Resistor_THT:R_Axial_DIN0204_L3.6mm_D1.6mm_P7.62mm_Horizontal
Changed lines of the file:
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@@
       (effects (font (size 1.27 1.27)) (justify left))
     )
-    (property "Footprint" "agausmann:R_Hybrid_SMD_THT" (id 2) (at 102.362 153.67 90)
+    (property "Footprint" "Resistor_THT:R_Axial_DIN0204_L3.6mm_D1.6mm_P7.62mm_Horizontal" (id 2) (at 102.362 153.67 90)
       (effects (font (size 1.27 1.27)) hide)
     )
@@
       (effects (font (size 1.27 1.27)) (justify left))
     )
-    (property "Footprint" "agausmann:R_Hybrid_SMD_THT" (id 2) (at 93.472 153.67 90)
+    (property "Footprint" "Resistor_THT:R_Axial_DIN0204_L3.6mm_D1.6mm_P7.62mm_Horizontal" (id 2) (at 93.472 153.67 90)
       (effects (font (size 1.27 1.27)) hide)
     )
@@
       (effects (font (size 1.27 1.27)) (justify left))
     )
-    (property "Footprint" "agausmann:R_Hybrid_SMD_THT" (id 2) (at 75.692 153.67 90)
+    (property "Footprint" "Resistor_THT:R_Axial_DIN0204_L3.6mm_D1.6mm_P7.62mm_Horizontal" (id 2) (at 75.692 153.67 90)
       (effects (font (size 1.27 1.27)) hide)
     )
@@
       (effects (font (size 1.27 1.27)) (justify left))
     )
-    (property "Footprint" "agausmann:R_Hybrid_SMD_THT" (id 2) (at 66.802 153.67 90)
+    (property "Footprint" "Resistor_THT:R_Axial_DIN0204_L3.6mm_D1.6mm_P7.62mm_Horizontal" (id 2) (at 66.802 153.67 90)
       (effects (font (size 1.27 1.27)) hide)
     )
@@
       (effects (font (size 1.27 1.27)) (justify left))
     )
-    (property "Footprint" "agausmann:R_Hybrid_SMD_THT" (id 2) (at 57.912 153.67 90)
+    (property "Footprint" "Resistor_THT:R_Axial_DIN0204_L3.6mm_D1.6mm_P7.62mm_Horizontal" (id 2) (at 57.912 153.67 90)
       (effects (font (size 1.27 1.27)) hide)
     )
@@
       (effects (font (size 1.27 1.27)) (justify left))
     )
-    (property "Footprint" "agausmann:R_Hybrid_SMD_THT" (id 2) (at 84.582 153.67 90)
+    (property "Footprint" "Resistor_THT:R_Axial_DIN0204_L3.6mm_D1.6mm_P7.62mm_Horizontal" (id 2) (at 84.582 153.67 90)
       (effects (font (size 1.27 1.27)) hide)
     )
